File: gas-sensor-simple/gas-sensor-simple.sch (KiCad schematic (older format))
At the start: 25 parts, among them J1 6-pin male, J2 6-pin female, J3 8-pin male, U1 MQ-8, U1 ads1x15, U10 MV5x3x, U11 MV5x3x, U2 MQ-4, U3 O2, U4 CO2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

Commit message: Schematic passes checks. Nearly complete. Need to sort out alert, addr and cs pins on digital side.
Parts:
- removed U3: O2, symbol MQxModule
- removed U4: CO2, symbol MQxModule
- removed U6: 7407, symbol 7407
- removed U?: BME280, symbol BME280
- added RN1: 4 x 100K, Resistors_THT:R_Array_SIP8, symbol R_Pack04_SIP
- added RV1: 10K, symbol POT_TRIM
- added TH1, TH2, TH3, TH4: 100K, symbol Thermistor
- added U12: LM393, symbol LM393
- added U15: BME280, symbol BME280
- added U3: CO2, symbol DFRobotCO2
- added U4: O2, symbol LinkSpriteO2
- added unit 2 of U6
- R1, R3, R5, R7: value R -> 140
- R2, R4, R6, R8: value R -> 160
- gave numbers to parts that had none: 1
- renumbered U1 to U13
Connections:
- net labels added: +3.3V, GND, GNDD
- net labels removed: VAA
- wire segments 102 -> 172
- no-connect marks 3 -> 6
Other:
- moved on the sheet: J3, U13, U14, U5B

Commit message: Tweaks to schematic. Add screen capture: schematic.png
Connections:
- net GNDA is gone; now on net GND: J2.2 (Pin_2), J3.3 (Pin_3), TH1.2, TH2.2, TH3.2, TH4.2, U15.1 (GND), U15.10 (GND), U15.5 (~CS~)
Other:
- note added: "Bionic Leaf CO2, O2, H2 and CH4 \ngas detector with digital interface"

Commit message: More tweaks. Find out how to fill background of components, so update bionicleaf.lib and schematic.
Connections:
- net GND: now also U13.2 (GND), U14.2 (GND)
- net at U13.5 (ADDR): now also J3.7 (Pin_7)
- net at U13.6 (ALERT): now also J3.8 (Pin_8)
Other:
- moved on the sheet: J1, J2, J3, R1, R2, R3, R4, R5, R6, R7, R8, RN1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
