File: gas-sensor-simple/gas-sensor-simple.kicad_pcb (KiCad board)
At the start: 2 copper layers, 91.4 x 99.1 mm, 43 parts, among them J1 2x5 pin, J2 2x5 socket, J3 2x5 pin, J4 1x2, J5 1x2, J6 1x2, J7 1x2, U1 MQ-8, U10 RG LED, U12 LM393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

Commit message: Version of boards that was sent for prototypes
Parts:
- added .: ., Pin_Headers:Pin_Header_Straight_2x04_Pitch2.54mm, F.Cu at (227.3, 124.5)
- added ..: ., Pin_Headers:Pin_Header_Straight_2x04_Pitch2.54mm, F.Cu at (232.4, 124.5)
- added ...: ,, Pin_Headers:Pin_Header_Straight_2x04_Pitch2.54mm, F.Cu at (237.5, 124.5)
- J1: value 2x5 pin -> RPi
- J2: value 2x5 socket -> digital header
- J3: value 2x5 pin -> digital header
- RN3: value 4x180 -> 4x150
- moved U15 94.1 mm to (199.4, 105.4), turned to 270 degrees
- moved J1 91.2 mm to (195.6, 53.3), turned to 270 degrees
- moved C4 88.8 mm to (200.7, 55.8), turned to 90 degrees
- moved C2 87.5 mm to (200.7, 60.2)
- moved C1 82.8 mm to (190.5, 60.2)
- moved C3 80.2 mm to (195.6, 62.2), turned to 90 degrees
- moved R10 75.0 mm to (191.8, 90.2), turned to 90 degrees
- moved U14 66.5 mm to (184.2, 77.5)
- moved U10 64.7 mm to (250.2, 127.0)
- moved RV1 64.1 mm to (241.3, 139.8)
- moved C8 63.8 mm to (179.1, 69.1)
- moved U9 63.8 mm to (250.2, 111.8)
- moved C9 63.8 mm to (184.2, 71.1), turned to 90 degrees
- moved U8 63.6 mm to (250.2, 96.5)
- moved U7 63.5 mm to (250.2, 81.3)
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Routing:
- net Net-(J1-Pad7): track 12.5 -> 60.3 mm
- net Net-(J2-Pad8): track 81.9 -> 42.0 mm
- net Net-(J1-Pad5): track 73.9 -> 113.1 mm
- net GNDD: track 97.8 -> 135.9 mm
- net Net-(J2-Pad10): track 74.6 -> 38.4 mm
- net VCC: track 269.4 -> 304.4 mm
- net Net-(J2-Pad6): track 78.0 -> 45.6 mm
- net Net-(J2-Pad4): track 80.4 -> 49.2 mm
- net Net-(J2-Pad9): track 49.8 -> 79.9 mm, vias 0 -> 1
- net Net-(R10-Pad1): track 36.0 -> 7.62 mm
- net Net-(RV1-Pad2): track 17.0 -> 41.0 mm
- net +3V3: track 114.9 -> 138.5 mm
- net Net-(J2-Pad7): track 47.6 -> 70.9 mm, vias 0 -> 1
- net GND: track 251.4 -> 272.5 mm
- net Net-(U3-Pad4): track 31.4 -> 49.1 mm
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Other:
- board size 91.4 x 99.1 mm -> 97.8 x 99.1 mm
- rule pad_to_mask_clearance: 0 -> 0.254
- board text added: "proto area"
- board text removed: "1.0"
- board text removed: "2017-11-14"
- board text removed: "Analog gas sensor and digital interface"
- board text removed: "Gas Sensor v1"
